Commit message: 更新go2描述文件

File: unitree_go2_ros2_function_pkg/src/go2_sim/urdf/go2_description.urdf (robot description, URDF)
Before this commit: robot go2_description, 29 links, 28 joints
Links:
- removed link base_link
- added link base, mass 6.921; collision box size=0.3762 0.0935 0.114; visual mesh filename=package://go2_description/dae/base.dae
- link radar: mass 0.01 -> 0
Joints:
- joint FL_hip_joint: parent base_link -> base
- joint FR_hip_joint: parent base_link -> base
- joint Head_upper_joint: parent base_link -> base
- joint RL_hip_joint: parent base_link -> base
- joint RR_hip_joint: parent base_link -> base
- joint imu_joint: parent base_link -> base
- joint radar_joint: parent base_link -> base

File: unitree_go2_ros2_function_pkg/src/go2_sim/xacro/gazebo.xacro (robot description, xacro)
@@ -29,10 +29,10 @@
         </plugin>
     </gazebo>
-    <!-- <gazebo>
-        <plugin filename="/opt/ros/humble/lib/libgazebo_ros_force.so name="gazebo_ros_force" " >
+    <gazebo>
+        <plugin filename="libgazebo_ros_force.so" name="gazebo_ros_force">
             <bodyName>trunk</bodyName>
             <topicName>/apply_force/trunk</topicName>
         </plugin>
-    </gazebo> -->
+    </gazebo>
     <gazebo reference="imu_link">
         <gravity>true</gravity>

File: unitree_go2_ros2_function_pkg/src/go2_sim/xacro/leg.xacro (robot description, xacro)
@@ -1,5 +1,5 @@
 <?xml version="1.0"?>
 <robot xmlns:xacro="http://www.ros.org/wiki/xacro">
-    <xacro:include filename="$(find go2_urdf)/xacro/transmission.xacro"/>
+    <xacro:include filename="$(find go2_description)/xacro/transmission.xacro"/>
     <xacro:macro name="leg" params="name mirror mirror_dae front_hind front_hind_dae">
         <joint name="${name}_hip_joint" type="revolute">
@@ -42,5 +42,5 @@
                 </xacro:if>
                 <geometry>
-                    <mesh filename="package://go2_urdf/meshes/hip.dae" scale="1 1 1"/>
+                    <mesh filename="package://go2_description/meshes/hip.dae" scale="1 1 1"/>
                 </geometry>
                 <!-- <material name="orange"/> -->
@@ -74,8 +74,8 @@
                 <geometry>
                     <xacro:if value="${mirror_dae == True}">
-                        <mesh filename="package://go2_urdf/meshes/thigh.dae" scale="1 1 1"/>
+                        <mesh filename="package://go2_description/meshes/thigh.dae" scale="1 1 1"/>
                     </xacro:if>
                     <xacro:if value="${mirror_dae == False}">
-                        <mesh filename="package://go2_urdf/meshes/thigh_mirror.dae" scale="1 1 1"/>
+                        <mesh filename="package://go2_description/meshes/thigh_mirror.dae" scale="1 1 1"/>
                     </xacro:if>
                 </geometry>
@@ -109,5 +109,5 @@
                 <origin rpy="0 0 0" xyz="0 0 0"/>
                 <geometry>
-                    <mesh filename="package://go2_urdf/meshes/calf.dae" scale="1 1 1"/>
+                    <mesh filename="package://go2_description/meshes/calf.dae" scale="1 1 1"/>
                 </geometry>
                 <!-- <material name="orange"/> -->

File: unitree_go2_ros2_function_pkg/src/go2_sim/xacro/robot.xacro (robot description, xacro)
@@ -2,9 +2,9 @@
 <robot name="go2" xmlns:xacro="http://www.ros.org/wiki/xacro">
     <xacro:arg name="DEBUG" default="false"/>
-    <xacro:include filename="$(find go2_urdf)/xacro/const.xacro"/>
-    <xacro:include filename="$(find go2_urdf)/xacro/materials.xacro"/>
-    <xacro:include filename="$(find go2_urdf)/xacro/leg.xacro"/>
-    <!-- <xacro:include filename="$(find go2_urdf)/xacro/stairs.xacro"/> -->
-    <xacro:include filename="$(find go2_urdf)/xacro/gazebo.xacro"/>
+    <xacro:include filename="$(find go2_description)/xacro/const.xacro"/>
+    <xacro:include filename="$(find go2_description)/xacro/materials.xacro"/>
+    <xacro:include filename="$(find go2_description)/xacro/leg.xacro"/>
+    <!-- <xacro:include filename="$(find go2_description)/xacro/stairs.xacro"/> -->
+    <xacro:include filename="$(find go2_description)/xacro/gazebo.xacro"/>
     <!-- <xacro:include filename="$(find go2_gazebo)/launch/stairs.urdf.xacro"/> -->
     <!-- <xacro:stairs stairs="15" xpos="0" ypos="0" zpos="0" /> -->
@@ -37,5 +37,5 @@
             <origin rpy="0 0 0" xyz="0 0 0"/>
             <geometry>
-                <mesh filename="package://go2_urdf/meshes/trunk.dae" scale="1 1 1"/>
+                <mesh filename="package://go2_description/meshes/trunk.dae" scale="1 1 1"/>
             </geometry>
             <!-- <material name="orange"/> -->

Commit message: 修复导航节点的bug

File: unitree_go2_ros2_function_pkg/src/go2_sim/urdf/go2_description.urdf (robot description, URDF)
Before this commit: robot go2_description, 29 links, 28 joints
Links:
- removed link radar
- added link go2_lidar, mass 0
Joints:
- removed joint radar_joint
- added joint go2_lidar_joint: type fixed, parent base, child go2_lidar, origin xyz=0.28945 0 -0.046825 rpy=0 2.8782 0, axis 0 0 0

Commit message: go2增加仿真描述文件

File: unitree_go2_ros2_function_pkg/src/go2_sim/urdf/go2_description.urdf (robot description, URDF)
Before this commit: robot go2_description, 29 links, 28 joints
Links:
- link FL_calf: geometry collision cylinder length=0.12 radius=0.012; visual mesh filename=package://go2_sim/dae/calf.dae
- link FL_foot: geometry collision sphere radius=0.022; visual mesh filename=package://go2_sim/dae/foot.dae
- link FL_hip: geometry collision cylinder length=0.04 radius=0.046; visual mesh filename=package://go2_sim/dae/hip.dae
- link FL_thigh: geometry collision box size=0.213 0.0245 0.034; visual mesh filename=package://go2_sim/dae/thigh.dae
- link FR_calf: geometry collision cylinder length=0.12 radius=0.013; visual mesh filename=package://go2_sim/dae/calf_mirror.dae
- link FR_foot: geometry collision sphere radius=0.022; visual mesh filename=package://go2_sim/dae/foot.dae
- link FR_hip: geometry collision cylinder length=0.04 radius=0.046; visual mesh filename=package://go2_sim/dae/hip.dae
- link FR_thigh: geometry collision box size=0.213 0.0245 0.034; visual mesh filename=package://go2_sim/dae/thigh_mirror.dae
- link RL_calf: geometry collision cylinder length=0.12 radius=0.013; visual mesh filename=package://go2_sim/dae/calf.dae
- link RL_foot: geometry collision sphere radius=0.022; visual mesh filename=package://go2_sim/dae/foot.dae
- link RL_hip: geometry collision cylinder length=0.04 radius=0.046; visual mesh filename=package://go2_sim/dae/hip.dae
- link RL_thigh: geometry collision box size=0.213 0.0245 0.034; visual mesh filename=package://go2_sim/dae/thigh.dae
- link RR_calf: geometry collision cylinder length=0.12 radius=0.013; visual mesh filename=package://go2_sim/dae/calf_mirror.dae
- link RR_foot: geometry collision sphere radius=0.022; visual mesh filename=package://go2_sim/dae/foot.dae
- link RR_hip: geometry collision cylinder length=0.04 radius=0.046; visual mesh filename=package://go2_sim/dae/hip.dae
- link RR_thigh: geometry collision box size=0.213 0.0245 0.034; visual mesh filename=package://go2_sim/dae/thigh_mirror.dae
- link base: geometry collision box size=0.3762 0.0935 0.114; visual mesh filename=package://go2_sim/dae/base.dae

File: unitree_go2_ros2_function_pkg/src/go2_sim/xacro/leg.xacro (robot description, xacro)
@@ -1,5 +1,5 @@
 <?xml version="1.0"?>
 <robot xmlns:xacro="http://www.ros.org/wiki/xacro">
-    <xacro:include filename="$(find go2_description)/xacro/transmission.xacro"/>
+    <xacro:include filename="$(find go2_sim)/xacro/transmission.xacro"/>
     <xacro:macro name="leg" params="name mirror mirror_dae front_hind front_hind_dae">
         <joint name="${name}_hip_joint" type="revolute">
@@ -42,5 +42,5 @@
                 </xacro:if>
                 <geometry>
-                    <mesh filename="package://go2_description/meshes/hip.dae" scale="1 1 1"/>
+                    <mesh filename="package://go2_sim/meshes/hip.dae" scale="1 1 1"/>
                 </geometry>
                 <!-- <material name="orange"/> -->
@@ -74,8 +74,8 @@
                 <geometry>
                     <xacro:if value="${mirror_dae == True}">
-                        <mesh filename="package://go2_description/meshes/thigh.dae" scale="1 1 1"/>
+                        <mesh filename="package://go2_sim/meshes/thigh.dae" scale="1 1 1"/>
                     </xacro:if>
                     <xacro:if value="${mirror_dae == False}">
-                        <mesh filename="package://go2_description/meshes/thigh_mirror.dae" scale="1 1 1"/>
+                        <mesh filename="package://go2_sim/meshes/thigh_mirror.dae" scale="1 1 1"/>
                     </xacro:if>
                 </geometry>
@@ -109,5 +109,5 @@
                 <origin rpy="0 0 0" xyz="0 0 0"/>
                 <geometry>
-                    <mesh filename="package://go2_description/meshes/calf.dae" scale="1 1 1"/>
+                    <mesh filename="package://go2_sim/meshes/calf.dae" scale="1 1 1"/>
                 </geometry>
                 <!-- <material name="orange"/> -->

File: unitree_go2_ros2_function_pkg/src/go2_sim/xacro/robot.xacro (robot description, xacro)
@@ -2,9 +2,9 @@
 <robot name="go2" xmlns:xacro="http://www.ros.org/wiki/xacro">
     <xacro:arg name="DEBUG" default="false"/>
-    <xacro:include filename="$(find go2_description)/xacro/const.xacro"/>
-    <xacro:include filename="$(find go2_description)/xacro/materials.xacro"/>
-    <xacro:include filename="$(find go2_description)/xacro/leg.xacro"/>
-    <!-- <xacro:include filename="$(find go2_description)/xacro/stairs.xacro"/> -->
-    <xacro:include filename="$(find go2_description)/xacro/gazebo.xacro"/>
+    <xacro:include filename="$(find go2_sim)/xacro/const.xacro"/>
+    <xacro:include filename="$(find go2_sim)/xacro/materials.xacro"/>
+    <xacro:include filename="$(find go2_sim)/xacro/leg.xacro"/>
+    <!-- <xacro:include filename="$(find go2_sim)/xacro/stairs.xacro"/> -->
+    <xacro:include filename="$(find go2_sim)/xacro/gazebo.xacro"/>
     <!-- <xacro:include filename="$(find go2_gazebo)/launch/stairs.urdf.xacro"/> -->
     <!-- <xacro:stairs stairs="15" xpos="0" ypos="0" zpos="0" /> -->
@@ -37,5 +37,5 @@
             <origin rpy="0 0 0" xyz="0 0 0"/>
             <geometry>
-                <mesh filename="package://go2_description/meshes/trunk.dae" scale="1 1 1"/>
+                <mesh filename="package://go2_sim/meshes/trunk.dae" scale="1 1 1"/>
             </geometry>
             <!-- <material name="orange"/> -->

Commit message: go2仿真模型导入+nav调试成功

File: unitree_go2_ros2_function_pkg/src/go2_sim/urdf/go2_description.urdf (robot description, URDF)
Before this commit: robot go2_description, 29 links, 28 joints
Links:
- added link l1_lidar, mass 0
- link go2_lidar: mass 0 -> 0.5; geometry collision cylinder length=0.07 radius=0.05; visual cylinder length=0.07 radius=0.05
Joints:
- added joint l1_lidar_joint: type fixed, parent base, child l1_lidar, origin xyz=0.28945 0 -0.046825 rpy=0 2.8782 0, axis 0 0 0
- joint go2_lidar_joint: axis 0 0 0 -> (none); origin xyz=0.28945 0 -0.046825 rpy=0 2.8782 0 -> xyz=0.171 0.0 0.1108 rpy=0 0 1.5708

Commit message: 传感器同步节点优化

File: unitree_go2_ros2_function_pkg/src/go2_sim/urdf/go2_description.urdf (robot description, URDF)
Before this commit: robot go2_description, 30 links, 29 joints
Links:
- added link camera_link
Joints:
- added joint d435_joint: type fixed, parent base, child camera_link, origin xyz=0.3 0.0 0.0608 rpy=0 0 0

Commit message: 1、更新传感器同步节点 2、更新配套脑机接口调试节点

File: unitree_go2_ros2_function_pkg/src/go2_sim/urdf/go2_description.urdf (robot description, URDF)
Before this commit: robot go2_description, 31 links, 30 joints
Links:
- removed link go2_lidar
- added link hesai_lidar, mass 0.5; collision cylinder length=0.07 radius=0.05; visual cylinder length=0.07 radius=0.05
Joints:
- removed joint go2_lidar_joint
- added joint hesai_lidar_joint: type fixed, parent base, child hesai_lidar, origin xyz=0.171 0.0 0.1108 rpy=0 0 1.5708
